Commit message: Commit with drone stand

File: urdf/frame.xacro (robot description, xacro)
@@ -6,7 +6,7 @@
 <link name="base_link">
   <inertial>
-    <origin xyz="1.9090327228285685e-16 0.01999999999999998 1.9090327228285685e-16" rpy="0 0 0"/>
-    <mass value="0.6812756051704826"/>
-    <inertia ixx="0.006887" iyy="0.013384" izz="0.006887" ixy="-0.0" iyz="-0.0" ixz="0.0"/>
+    <origin xyz="5.361940941515797e-15 -0.006931498212032427 1.0942736615338362e-16" rpy="0 0 0"/>
+    <mass value="0.950824254848482"/>
+    <inertia ixx="0.010991" iyy="0.017094" izz="0.010991" ixy="0.0" iyz="0.0" ixz="0.0"/>
   </inertial>
   <visual>
@@ -24,5 +24,5 @@
   </collision>
 </link>
-<link name="arm_v2__2__1">
+<link name="arm_7_1">
   <inertial>
     <origin xyz="-0.08302889455495802 -2.527437287236367e-11 -0.0973299825380552" rpy="0 0 0"/>
@@ -33,5 +33,5 @@
     <origin xyz="0.055 -0.02 0.2" rpy="0 0 0"/>
     <geometry>
-      <mesh filename="file://$(find frame_description)/meshes/arm_v2__2__1.stl" scale="0.001 0.001 0.001"/>
+      <mesh filename="file://$(find frame_description)/meshes/arm_7_1.stl" scale="0.001 0.001 0.001"/>
     </geometry>
     <material name="silver"/>
@@ -40,9 +40,9 @@
     <origin xyz="0.055 -0.02 0.2" rpy="0 0 0"/>
     <geometry>
-      <mesh filename="file://$(find frame_description)/meshes/arm_v2__2__1.stl" scale="0.001 0.001 0.001"/>
-    </geometry>
-  </collision>
-</link>
-<link name="arm_1_1">
+      <mesh filename="file://$(find frame_description)/meshes/arm_7_1.stl" scale="0.001 0.001 0.001"/>
+    </geometry>
+  </collision>
+</link>
+<link name="arm_8_1">
   <inertial>
     <origin xyz="-0.0973299825380552 2.527436940291672e-11 -0.08302889455495804" rpy="0 0 0"/>
@@ -53,5 +53,5 @@
     <origin xyz="0.2 -0.02 0.055" rpy="0 0 0"/>
     <geometry>
-      <mesh filename="file://$(find frame_description)/meshes/arm_1_1.stl" scale="0.001 0.001 0.001"/>
+      <mesh filename="file://$(find frame_description)/meshes/arm_8_1.stl" scale="0.001 0.001 0.001"/>
     </geometry>
     <material name="silver"/>
@@ -60,9 +60,9 @@
     <origin xyz="0.2 -0.02 0.055" rpy="0 0 0"/>
     <geometry>
-      <mesh filename="file://$(find frame_description)/meshes/arm_1_1.stl" scale="0.001 0.001 0.001"/>
-    </geometry>
-  </collision>
-</link>
-<link name="arm_v2__7__1">
+      <mesh filename="file://$(find frame_description)/meshes/arm_8_1.stl" scale="0.001 0.001 0.001"/>
+    </geometry>
+  </collision>
+</link>
+<link name="arm_6_1">
   <inertial>
     <origin xyz="0.0973299825380552 2.5274376341810623e-11 0.08302889455495804" rpy="0 0 0"/>
@@ -73,5 +73,5 @@
     <origin xyz="-0.2 -0.02 -0.055" rpy="0 0 0"/>
     <geometry>
-      <mesh filename="file://$(find frame_description)/meshes/arm_v2__7__1.stl" scale="0.001 0.001 0.001"/>
+      <mesh filename="file://$(find frame_description)/meshes/arm_6_1.stl" scale="0.001 0.001 0.001"/>
     </geometry>
     <material name="silver"/>
@@ -80,9 +80,9 @@
     <origin xyz="-0.2 -0.02 -0.055" rpy="0 0 0"/>
     <geometry>
-      <mesh filename="file://$(find frame_description)/meshes/arm_v2__7__1.stl" scale="0.001 0.001 0.001"/>
-    </geometry>
-  </collision>
-</link>
-<link name="arm_v2__4__1">
+      <mesh filename="file://$(find frame_description)/meshes/arm_6_1.stl" scale="0.001 0.001 0.001"/>
+    </geometry>
+  </collision>
+</link>
+<link name="arm_5_1">
   <inertial>
     <origin xyz="0.08302889455495802 -2.527437287236367e-11 0.0973299825380552" rpy="0 0 0"/>
@@ -93,5 +93,5 @@
     <origin xyz="-0.055 -0.02 -0.2" rpy="0 0 0"/>
     <geometry>
-      <mesh filename="file://$(find frame_description)/meshes/arm_v2__4__1.stl" scale="0.001 0.001 0.001"/>
+      <mesh filename="file://$(find frame_description)/meshes/arm_5_1.stl" scale="0.001 0.001 0.001"/>
     </geometry>
     <material name="silver"/>
@@ -100,9 +100,9 @@
     <origin xyz="-0.055 -0.02 -0.2" rpy="0 0 0"/>
     <geometry>
-      <mesh filename="file://$(find frame_description)/meshes/arm_v2__4__1.stl" scale="0.001 0.001 0.001"/>
-    </geometry>
-  </collision>
-</link>
-<link name="arm_v2__5__1">
+      <mesh filename="file://$(find frame_description)/meshes/arm_5_1.stl" scale="0.001 0.001 0.001"/>
+    </geometry>
+  </collision>
+</link>
+<link name="arm_4_1">
   <inertial>
     <origin xyz="0.0973299825380552 -2.527437287236367e-11 -0.08302889455495804" rpy="0 0 0"/>
@@ -113,5 +113,5 @@
     <origin xyz="-0.2 -0.02 0.055" rpy="0 0 0"/>
     <geometry>
-      <mesh filename="file://$(find frame_description)/meshes/arm_v2__5__1.stl" scale="0.001 0.001 0.001"/>
+      <mesh filename="file://$(find frame_description)/meshes/arm_4_1.stl" scale="0.001 0.001 0.001"/>
     </geometry>
     <material name="silver"/>
@@ -120,9 +120,9 @@
     <origin xyz="-0.2 -0.02 0.055" rpy="0 0 0"/>
     <geometry>
-      <mesh filename="file://$(find frame_description)/meshes/arm_v2__5__1.stl" scale="0.001 0.001 0.001"/>
-    </geometry>
-  </collision>
-</link>
-<link name="arm_v2__6__1">
+      <mesh filename="file://$(find frame_description)/meshes/arm_4_1.stl" scale="0.001 0.001 0.001"/>
+    </geometry>
+  </collision>
+</link>
+<link name="arm_3_1">
   <inertial>
     <origin xyz="0.08302889455495802 2.527436940291672e-11 -0.0973299825380552" rpy="0 0 0"/>
@@ -133,5 +133,5 @@
     <origin xyz="-0.055 -0.02 0.2" rpy="0 0 0"/>
     <geometry>
-      <mesh filename="file://$(find frame_description)/meshes/arm_v2__6__1.stl" scale="0.001 0.001 0.001"/>
+      <mesh filename="file://$(find frame_description)/meshes/arm_3_1.stl" scale="0.001 0.001 0.001"/>
     </geometry>
     <material name="silver"/>
@@ -140,9 +140,9 @@
     <origin xyz="-0.055 -0.02 0.2" rpy="0 0 0"/>
     <geometry>
-      <mesh filename="file://$(find frame_description)/meshes/arm_v2__6__1.stl" scale="0.001 0.001 0.001"/>
-    </geometry>
-  </collision>
-</link>
-<link name="arm_v2__1__1">
+      <mesh filename="file://$(find frame_description)/meshes/arm_3_1.stl" scale="0.001 0.001 0.001"/>
+    </geometry>
+  </collision>
+</link>
+<link name="arm_2_1">
   <inertial>
     <origin xyz="-0.09732998253804703 -2.5274383280704527e-11 0.08302889455496792" rpy="0 0 0"/>
@@ -153,5 +153,5 @@
     <origin xyz="0.2 -0.02 -0.055" rpy="0 0 0"/>
     <geometry>
-      <mesh filename="file://$(find frame_description)/meshes/arm_v2__1__1.stl" scale="0.001 0.001 0.001"/>
+      <mesh filename="file://$(find frame_description)/meshes/arm_2_1.stl" scale="0.001 0.001 0.001"/>
     </geometry>
     <material name="silver"/>
@@ -160,11 +160,11 @@
     <origin xyz="0.2 -0.02 -0.055" rpy="0 0 0"/>
     <geometry>
-      <mesh filename="file://$(find frame_description)/meshes/arm_v2__1__1.stl" scale="0.001 0.001 0.001"/>
-    </geometry>
-  </collision>
-</link>
-<link name="arm_v2__3__1">
-  <inertial>
-    <origin xyz="-0.08302889455495796 2.5278622944879814e-11 0.0973299825380552" rpy="0 0 0"/>
+      <mesh filename="file://$(find frame_description)/meshes/arm_2_1.stl" scale="0.001 0.001 0.001"/>
+    </geometry>
+  </collision>
+</link>
+<link name="arm_1_1">
+  <inertial>
+    <origin xyz="-0.08302889455495796 2.5278522330918207e-11 0.09732998253805508" rpy="0 0 0"/>
     <mass value="0.15422742956922936"/>
     <inertia ixx="0.000389" iyy="0.000929" izz="0.0006" ixy="0.0" iyz="-0.0" ixz="0.000277"/>
@@ -173,5 +173,5 @@
     <origin xyz="0.055 -0.02 -0.2" rpy="0 0 0"/>
     <geometry>
-      <mesh filename="file://$(find frame_description)/meshes/arm_v2__3__1.stl" scale="0.001 0.001 0.001"/>
+      <mesh filename="file://$(find frame_description)/meshes/arm_1_1.stl" scale="0.001 0.001 0.001"/>
     </geometry>
     <material name="silver"/>
@@ -180,9 +180,9 @@
     <origin xyz="0.055 -0.02 -0.2" rpy="0 0 0"/>
     <geometry>
-      <mesh filename="file://$(find frame_description)/meshes/arm_v2__3__1.stl" scale="0.001 0.001 0.001"/>
-    </geometry>
-  </collision>
-</link>
-<link name="holder_v1_1">
+      <mesh filename="file://$(find frame_description)/meshes/arm_1_1.stl" scale="0.001 0.001 0.001"/>
+    </geometry>
+  </collision>
+</link>
+<link name="holder_4_1">
   <inertial>
     <origin xyz="0.0012743502456399602 -1.933707013956898e-11 -0.016274350245639946" rpy="0 0 0"/>
@@ -193,5 +193,5 @@
     <origin xyz="0.2 -0.02 -0.215" rpy="0 0 0"/>
     <geometry>
-      <mesh filename="file://$(find frame_description)/meshes/holder_v1_1.stl" scale="0.001 0.001 0.001"/>
+      <mesh filename="file://$(find frame_description)/meshes/holder_4_1.stl" scale="0.001 0.001 0.001"/>
     </geometry>
     <material name="silver"/>
@@ -200,9 +200,9 @@
     <origin xyz="0.2 -0.02 -0.215" rpy="0 0 0"/>
     <geometry>
-      <mesh filename="file://$(find frame_description)/meshes/holder_v1_1.stl" scale="0.001 0.001 0.001"/>
-    </geometry>
-  </collision>
-</link>
-<link name="holder_v1_1">
+      <mesh filename="file://$(find frame_description)/meshes/holder_4_1.stl" scale="0.001 0.001 0.001"/>
+    </geometry>
+  </collision>
+</link>
+<link name="holder_4_1">
   <inertial>
     <origin xyz="0.016274350245639946 -1.933707013956898e-11 -0.0012743502456399602" rpy="0 0 0"/>
@@ -213,5 +213,5 @@
     <origin xyz="0.215 -0.02 -0.2" rpy="0 0 0"/>
     <geometry>
-      <mesh filename="file://$(find frame_description)/meshes/holder_v1_1.stl" scale="0.001 0.001 0.001"/>
+      <mesh filename="file://$(find frame_description)/meshes/holder_4_1.stl" scale="0.001 0.001 0.001"/>
     </geometry>
     <material name="silver"/>
@@ -220,9 +220,9 @@
     <origin xyz="0.215 -0.02 -0.2" rpy="0 0 0"/>
     <geometry>
-      <mesh filename="file://$(find frame_description)/meshes/holder_v1_1.stl" scale="0.001 0.001 0.001"/>
-    </geometry>
-  </collision>
-</link>
-<link name="holder_v1__2__1">
+      <mesh filename="file://$(find frame_description)/meshes/holder_4_1.stl" scale="0.001 0.001 0.001"/>
+    </geometry>
+  </collision>
+</link>
+<link name="holder_3_1">
   <inertial>
     <origin xyz="0.01627435024563989 3.173676564605099e-10 0.0012743502456399047" rpy="0 0 0"/>
@@ -233,5 +233,5 @@
     <origin xyz="0.215 -0.02 0.2" rpy="0 0 0"/>
     <geometry>
-      <mesh filename="file://$(find frame_description)/meshes/holder_v1__2__1.stl" scale="0.001 0.001 0.001"/>
+      <mesh filename="file://$(find frame_description)/meshes/holder_3_1.stl" scale="0.001 0.001 0.001"/>
     </geometry>
     <material name="silver"/>
@@ -240,9 +240,9 @@
     <origin xyz="0.215 -0.02 0.2" rpy="0 0 0"/>
     <geometry>
-      <mesh filename="file://$(find frame_description)/meshes/holder_v1__2__1.stl" scale="0.001 0.001 0.001"/>
-    </geometry>
-  </collision>
-</link>
-<link name="holder_v1__2__1">
+      <mesh filename="file://$(find frame_description)/meshes/holder_3_1.stl" scale="0.001 0.001 0.001"/>
+    </geometry>
+  </collision>
+</link>
+<link name="holder_3_1">
   <inertial>
     <origin xyz="0.0012743502456399047 3.173676564605099e-10 0.01627435024563989" rpy="0 0 0"/>
@@ -253,5 +253,5 @@
     <origin xyz="0.2 -0.02 0.215" rpy="0 0 0"/>
     <geometry>
-      <mesh filename="file://$(find frame_description)/meshes/holder_v1__2__1.stl" scale="0.001 0.001 0.001"/>
+      <mesh filename="file://$(find frame_description)/meshes/holder_3_1.stl" scale="0.001 0.001 0.001"/>
     </geometry>
     <material name="silver"/>
@@ -260,9 +260,9 @@
     <origin xyz="0.2 -0.02 0.215" rpy="0 0 0"/>
     <geometry>
-      <mesh filename="file://$(find frame_description)/meshes/holder_v1__2__1.stl" scale="0.001 0.001 0.001"/>
-    </geometry>
-  </collision>
-</link>
-<link name="holder_v1__3__1">
+      <mesh filename="file://$(find frame_description)/meshes/holder_3_1.stl" scale="0.001 0.001 0.001"/>
+    </geometry>
+  </collision>
+</link>
+<link name="holder_2_1">
   <inertial>
     <origin xyz="-0.0012743502456399047 -1.9344432306001025e-11 0.01627435024563989" rpy="0 0 0"/>
@@ -273,5 +273,5 @@
     <origin xyz="-0.2 -0.02 0.215" rpy="0 0 0"/>
     <geometry>
-      <mesh filename="file://$(find frame_description)/meshes/holder_v1__3__1.stl" scale="0.001 0.001 0.001"/>
+      <mesh filename="file://$(find frame_description)/meshes/holder_2_1.stl" scale="0.001 0.001 0.001"/>
     </geometry>
     <material name="silver"/>
@@ -280,9 +280,9 @@
     <origin xyz="-0.2 -0.02 0.215" rpy="0 0 0"/>
     <geometry>
-      <mesh filename="file://$(find frame_description)/meshes/holder_v1__3__1.stl" scale="0.001 0.001 0.001"/>
-    </geometry>
-  </collision>
-</link>
-<link name="holder_v1__3__1">
+      <mesh filename="file://$(find frame_description)/meshes/holder_2_1.stl" scale="0.001 0.001 0.001"/>
+    </geometry>
+  </collision>
+</link>
+<link name="holder_2_1">
   <inertial>
     <origin xyz="-0.01627435024563989 -1.9344432306001025e-11 0.0012743502456399047" rpy="0 0 0"/>
@@ -293,5 +293,5 @@
     <origin xyz="-0.215 -0.02 0.2" rpy="0 0 0"/>
     <geometry>
-      <mesh filename="file://$(find frame_description)/meshes/holder_v1__3__1.stl" scale="0.001 0.001 0.001"/>
+      <mesh filename="file://$(find frame_description)/meshes/holder_2_1.stl" scale="0.001 0.001 0.001"/>
     </geometry>
     <material name="silver"/>
@@ -300,9 +300,9 @@
     <origin xyz="-0.215 -0.02 0.2" rpy="0 0 0"/>
     <geometry>
-      <mesh filename="file://$(find frame_description)/meshes/holder_v1__3__1.stl" scale="0.001 0.001 0.001"/>
-    </geometry>
-  </collision>
-</link>
-<link name="holder_v1__1__1">
+      <mesh filename="file://$(find frame_description)/meshes/holder_2_1.stl" scale="0.001 0.001 0.001"/>
+    </geometry>
+  </collision>
+</link>
+<link name="holder_1_1">
   <inertial>
     <origin xyz="-0.01627435024563989 -1.9344414958766265e-11 -0.0012743502456399047" rpy="0 0 0"/>
@@ -313,5 +313,5 @@
     <origin xyz="-0.215 -0.02 -0.2" rpy="0 0 0"/>
     <geometry>
-      <mesh filename="file://$(find frame_description)/meshes/holder_v1__1__1.stl" scale="0.001 0.001 0.001"/>
+      <mesh filename="file://$(find frame_description)/meshes/holder_1_1.stl" scale="0.001 0.001 0.001"/>
     </geometry>
     <material name="silver"/>
@@ -320,9 +320,9 @@
     <origin xyz="-0.215 -0.02 -0.2" rpy="0 0 0"/>
     <geometry>
-      <mesh filename="file://$(find frame_description)/meshes/holder_v1__1__1.stl" scale="0.001 0.001 0.001"/>
-    </geometry>
-  </collision>
-</link>
-<link name="holder_v1__1__1">
+      <mesh filename="file://$(find frame_description)/meshes/holder_1_1.stl" scale="0.001 0.001 0.001"/>
+    </geometry>
+  </collision>
+</link>
+<link name="holder_1_1">
   <inertial>
     <origin xyz="-0.0012743502456399047 -1.9344414958766265e-11 -0.01627435024563989" rpy="0 0 0"/>
@@ -333,5 +333,5 @@
     <origin xyz="-0.2 -0.02 -0.215" rpy="0 0 0"/>
     <geometry>
-      <mesh filename="file://$(find frame_description)/meshes/holder_v1__1__1.stl" scale="0.001 0.001 0.001"/>
+      <mesh filename="file://$(find frame_description)/meshes/holder_1_1.stl" scale="0.001 0.001 0.001"/>
     </geometry>
     <material name="silver"/>
@@ -340,9 +340,9 @@
     <origin xyz="-0.2 -0.02 -0.215" rpy="0 0 0"/>
     <geometry>
-      <mesh filename="file://$(find frame_description)/meshes/holder_v1__1__1.stl" scale="0.001 0.001 0.001"/>
-    </geometry>
-  </collision>
-</link>
-<link name="bldc_v2__2__1">
+      <mesh filename="file://$(find frame_description)/meshes/holder_1_1.stl" scale="0.001 0.001 0.001"/>
+    </geometry>
+  </collision>
+</link>
+<link name="bldc_8_1">
   <inertial>
     <origin xyz="-9.850613495537841e-06 0.012072048037910045 2.6988692206020293e-05" rpy="0 0 0"/>
@@ -353,5 +353,5 @@
     <origin xyz="-0.2 -0.04 -0.2" rpy="0 0 0"/>
     <geometry>
-      <mesh filename="file://$(find frame_description)/meshes/bldc_v2__2__1.stl" scale="0.001 0.001 0.001"/>
+      <mesh filename="file://$(find frame_description)/meshes/bldc_8_1.stl" scale="0.001 0.001 0.001"/>
     </geometry>
     <material name="silver"/>
@@ -360,9 +360,9 @@
     <origin xyz="-0.2 -0.04 -0.2" rpy="0 0 0"/>
     <geometry>
-      <mesh filename="file://$(find frame_description)/meshes/bldc_v2__2__1.stl" scale="0.001 0.001 0.001"/>
-    </geometry>
-  </collision>
-</link>
-<link name="bldc_v2__1__1">
+      <mesh filename="file://$(find frame_description)/meshes/bldc_8_1.stl" scale="0.001 0.001 0.001"/>
+    </geometry>
+  </collision>
+</link>
+<link name="bldc_7_1">
   <inertial>
     <origin xyz="2.6989159021245657e-05 0.012072048037909955 9.851740487398786e-06" rpy="0 0 0"/>
@@ -373,5 +373,5 @@
     <origin xyz="-0.2 -0.04 0.2" rpy="0 0 0"/>
     <geometry>
-      <mesh filename="file://$(find frame_description)/meshes/bldc_v2__1__1.stl" scale="0.001 0.001 0.001"/>
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