Commit message: added virtual links

File: urdf/materials.xacro (robot description, xacro)
@@ -4,3 +4,12 @@
   <color rgba="0.700 0.700 0.700 1.000"/>
 </material>
+<material name="black">
+  <color rgba="0.000 0.000 0.000 1.000"/>
+</material>
+<material name="red">
+  <color rgba="1.000 0.000 0.000 1.000"/>
+</material>
+<material name="transparent">
+  <color rgba="0.000 0.000 0.000 0.000"/>
+</material>
 </robot>
