Commit message: changed joint limits

File: urdf/drone_frame.xacro (robot description, xacro)
@@ -1,7 +1,7 @@
 <?xml version="1.0" ?>
-<robot name="frame" xmlns:xacro="http://www.ros.org/wiki/xacro">
-<xacro:include filename="$(find frame_description)/urdf/materials.xacro" />
-<xacro:include filename="$(find frame_description)/urdf/frame.ros2control" />
-<xacro:include filename="$(find frame_description)/urdf/frame.gazebo" />
+<robot name="drone_frame" xmlns:xacro="http://www.ros.org/wiki/xacro">
+<xacro:include filename="$(find drone_frame_description)/urdf/materials.xacro" />
+<xacro:include filename="$(find drone_frame_description)/urdf/drone_frame.ros2control" />
+<xacro:include filename="$(find drone_frame_description)/urdf/drone_frame.gazebo" />
 <link name="base_link">
   <inertial>
@@ -13,5 +13,5 @@
     <origin xyz="0 0 0" rpy="0 0 0"/>
     <geometry>
-      <mesh filename="file://$(find frame_description)/meshes/base_link.stl" scale="0.001 0.001 0.001"/>
+      <mesh filename="file://$(find drone_frame_description)/meshes/base_link.stl" scale="0.001 0.001 0.001"/>
     </geometry>
     <material name="silver"/>
@@ -20,5 +20,5 @@
     <origin xyz="0 0 0" rpy="0 0 0"/>
     <geometry>
-      <mesh filename="file://$(find frame_description)/meshes/base_link.stl" scale="0.001 0.001 0.001"/>
+      <mesh filename="file://$(find drone_frame_description)/meshes/base_link.stl" scale="0.001 0.001 0.001"/>
     </geometry>
   </collision>
@@ -33,5 +33,5 @@
     <origin xyz="0.055 -0.02 0.2" rpy="0 0 0"/>
     <geometry>
-      <mesh filename="file://$(find frame_description)/meshes/arm_7_1.stl" scale="0.001 0.001 0.001"/>
+      <mesh filename="file://$(find drone_frame_description)/meshes/arm_7_1.stl" scale="0.001 0.001 0.001"/>
     </geometry>
     <material name="silver"/>
@@ -40,5 +40,5 @@
     <origin xyz="0.055 -0.02 0.2" rpy="0 0 0"/>
     <geometry>
-      <mesh filename="file://$(find frame_description)/meshes/arm_7_1.stl" scale="0.001 0.001 0.001"/>
+      <mesh filename="file://$(find drone_frame_description)/meshes/arm_7_1.stl" scale="0.001 0.001 0.001"/>
     </geometry>
   </collision>
@@ -53,5 +53,5 @@
     <origin xyz="0.2 -0.02 0.055" rpy="0 0 0"/>
     <geometry>
-      <mesh filename="file://$(find frame_description)/meshes/arm_8_1.stl" scale="0.001 0.001 0.001"/>
+      <mesh filename="file://$(find drone_frame_description)/meshes/arm_8_1.stl" scale="0.001 0.001 0.001"/>
     </geometry>
     <material name="silver"/>
@@ -60,5 +60,5 @@
     <origin xyz="0.2 -0.02 0.055" rpy="0 0 0"/>
     <geometry>
-      <mesh filename="file://$(find frame_description)/meshes/arm_8_1.stl" scale="0.001 0.001 0.001"/>
+      <mesh filename="file://$(find drone_frame_description)/meshes/arm_8_1.stl" scale="0.001 0.001 0.001"/>
     </geometry>
   </collision>
@@ -66,5 +66,5 @@
 <link name="arm_6_1">
   <inertial>
-    <origin xyz="0.0973299825380552 2.5274376341810623e-11 0.08302889455495804" rpy="0 0 0"/>
+    <origin xyz="0.09732998253805486 2.5274376341810623e-11 0.08302889455495802" rpy="0 0 0"/>
     <mass value="0.15422742956922936"/>
     <inertia ixx="0.0006" iyy="0.000929" izz="0.000389" ixy="-0.0" iyz="-0.0" ixz="-0.000277"/>
@@ -73,5 +73,5 @@
     <origin xyz="-0.2 -0.02 -0.055" rpy="0 0 0"/>
     <geometry>
-      <mesh filename="file://$(find frame_description)/meshes/arm_6_1.stl" scale="0.001 0.001 0.001"/>
+      <mesh filename="file://$(find drone_frame_description)/meshes/arm_6_1.stl" scale="0.001 0.001 0.001"/>
     </geometry>
     <material name="silver"/>
@@ -80,5 +80,5 @@
     <origin xyz="-0.2 -0.02 -0.055" rpy="0 0 0"/>
     <geometry>
-      <mesh filename="file://$(find frame_description)/meshes/arm_6_1.stl" scale="0.001 0.001 0.001"/>
+      <mesh filename="file://$(find drone_frame_description)/meshes/arm_6_1.stl" scale="0.001 0.001 0.001"/>
     </geometry>
   </collision>
@@ -93,5 +93,5 @@
     <origin xyz="-0.055 -0.02 -0.2" rpy="0 0 0"/>
     <geometry>
-      <mesh filename="file://$(find frame_description)/meshes/arm_5_1.stl" scale="0.001 0.001 0.001"/>
+      <mesh filename="file://$(find drone_frame_description)/meshes/arm_5_1.stl" scale="0.001 0.001 0.001"/>
     </geometry>
     <material name="silver"/>
@@ -100,5 +100,5 @@
     <origin xyz="-0.055 -0.02 -0.2" rpy="0 0 0"/>
     <geometry>
-      <mesh filename="file://$(find frame_description)/meshes/arm_5_1.stl" scale="0.001 0.001 0.001"/>
+      <mesh filename="file://$(find drone_frame_description)/meshes/arm_5_1.stl" scale="0.001 0.001 0.001"/>
     </geometry>
   </collision>
@@ -113,5 +113,5 @@
     <origin xyz="-0.2 -0.02 0.055" rpy="0 0 0"/>
     <geometry>
-      <mesh filename="file://$(find frame_description)/meshes/arm_4_1.stl" scale="0.001 0.001 0.001"/>
+      <mesh filename="file://$(find drone_frame_description)/meshes/arm_4_1.stl" scale="0.001 0.001 0.001"/>
     </geometry>
     <material name="silver"/>
@@ -120,5 +120,5 @@
     <origin xyz="-0.2 -0.02 0.055" rpy="0 0 0"/>
     <geometry>
-      <mesh filename="file://$(find frame_description)/meshes/arm_4_1.stl" scale="0.001 0.001 0.001"/>
+      <mesh filename="file://$(find drone_frame_description)/meshes/arm_4_1.stl" scale="0.001 0.001 0.001"/>
     </geometry>
   </collision>
@@ -133,5 +133,5 @@
     <origin xyz="-0.055 -0.02 0.2" rpy="0 0 0"/>
     <geometry>
-      <mesh filename="file://$(find frame_description)/meshes/arm_3_1.stl" scale="0.001 0.001 0.001"/>
+      <mesh filename="file://$(find drone_frame_description)/meshes/arm_3_1.stl" scale="0.001 0.001 0.001"/>
     </geometry>
     <material name="silver"/>
@@ -140,5 +140,5 @@
     <origin xyz="-0.055 -0.02 0.2" rpy="0 0 0"/>
     <geometry>
-      <mesh filename="file://$(find frame_description)/meshes/arm_3_1.stl" scale="0.001 0.001 0.001"/>
+      <mesh filename="file://$(find drone_frame_description)/meshes/arm_3_1.stl" scale="0.001 0.001 0.001"/>
     </geometry>
   </collision>
@@ -146,5 +146,5 @@
 <link name="arm_2_1">
   <inertial>
-    <origin xyz="-0.09732998253804703 -2.5274383280704527e-11 0.08302889455496792" rpy="0 0 0"/>
+    <origin xyz="-0.09732998253804709 -2.5269421971563233e-11 0.08302889455496792" rpy="0 0 0"/>
     <mass value="0.15422742956922936"/>
     <inertia ixx="0.0006" iyy="0.000929" izz="0.000389" ixy="-0.0" iyz="0.0" ixz="0.000277"/>
@@ -153,5 +153,5 @@
     <origin xyz="0.2 -0.02 -0.055" rpy="0 0 0"/>
     <geometry>
-      <mesh filename="file://$(find frame_description)/meshes/arm_2_1.stl" scale="0.001 0.001 0.001"/>
+      <mesh filename="file://$(find drone_frame_description)/meshes/arm_2_1.stl" scale="0.001 0.001 0.001"/>
     </geometry>
     <material name="silver"/>
@@ -160,5 +160,5 @@
     <origin xyz="0.2 -0.02 -0.055" rpy="0 0 0"/>
     <geometry>
-      <mesh filename="file://$(find frame_description)/meshes/arm_2_1.stl" scale="0.001 0.001 0.001"/>
+      <mesh filename="file://$(find drone_frame_description)/meshes/arm_2_1.stl" scale="0.001 0.001 0.001"/>
     </geometry>
   </collision>
@@ -166,5 +166,5 @@
 <link name="arm_1_1">
   <inertial>
-    <origin xyz="-0.08302889455495796 2.5278522330918207e-11 0.09732998253805508" rpy="0 0 0"/>
+    <origin xyz="-0.08302889455495796 2.5278622944879814e-11 0.0973299825380552" rpy="0 0 0"/>
     <mass value="0.15422742956922936"/>
     <inertia ixx="0.000389" iyy="0.000929" izz="0.0006" ixy="0.0" iyz="-0.0" ixz="0.000277"/>
@@ -173,5 +173,5 @@
     <origin xyz="0.055 -0.02 -0.2" rpy="0 0 0"/>
     <geometry>
-      <mesh filename="file://$(find frame_description)/meshes/arm_1_1.stl" scale="0.001 0.001 0.001"/>
+      <mesh filename="file://$(find drone_frame_description)/meshes/arm_1_1.stl" scale="0.001 0.001 0.001"/>
     </geometry>
     <material name="silver"/>
@@ -180,5 +180,5 @@
     <origin xyz="0.055 -0.02 -0.2" rpy="0 0 0"/>
     <geometry>
-      <mesh filename="file://$(find frame_description)/meshes/arm_1_1.stl" scale="0.001 0.001 0.001"/>
+      <mesh filename="file://$(find drone_frame_description)/meshes/arm_1_1.stl" scale="0.001 0.001 0.001"/>
     </geometry>
   </collision>
@@ -186,12 +186,12 @@
 <link name="holder_4_1">
   <inertial>
-    <origin xyz="0.0012743502456399602 -1.933707013956898e-11 -0.016274350245639946" rpy="0 0 0"/>
+    <origin xyz="0.0012743502456467604 -1.6835240493340287e-10 -0.0162743502456395" rpy="0 0 0"/>
     <mass value="0.545696208866394"/>
-    <inertia ixx="0.00016" iyy="0.000161" izz="0.00016" ixy="-0.0" iyz="0.0" ixz="-1e-06"/>
+    <inertia ixx="0.00016" iyy="0.000161" izz="0.00016" ixy="-0.0" iyz="-0.0" ixz="-1e-06"/>
   </inertial>
   <visual>
     <origin xyz="0.2 -0.02 -0.215" rpy="0 0 0"/>
     <geometry>
-      <mesh filename="file://$(find frame_description)/meshes/holder_4_1.stl" scale="0.001 0.001 0.001"/>
+      <mesh filename="file://$(find drone_frame_description)/meshes/holder_4_1.stl" scale="0.001 0.001 0.001"/>
     </geometry>
     <material name="silver"/>
@@ -200,5 +200,5 @@
     <origin xyz="0.2 -0.02 -0.215" rpy="0 0 0"/>
     <geometry>
-      <mesh filename="file://$(find frame_description)/meshes/holder_4_1.stl" scale="0.001 0.001 0.001"/>
+      <mesh filename="file://$(find drone_frame_description)/meshes/holder_4_1.stl" scale="0.001 0.001 0.001"/>
     </geometry>
   </collision>
@@ -206,12 +206,12 @@
 <link name="holder_4_1">
   <inertial>
-    <origin xyz="0.016274350245639946 -1.933707013956898e-11 -0.0012743502456399602" rpy="0 0 0"/>
+    <origin xyz="0.016274350245646746 -1.6835240493340287e-10 -0.0012743502456395162" rpy="0 0 0"/>
     <mass value="0.545696208866394"/>
-    <inertia ixx="0.00016" iyy="0.000161" izz="0.00016" ixy="-0.0" iyz="0.0" ixz="-1e-06"/>
+    <inertia ixx="0.00016" iyy="0.000161" izz="0.00016" ixy="-0.0" iyz="-0.0" ixz="-1e-06"/>
   </inertial>
   <visual>
     <origin xyz="0.215 -0.02 -0.2" rpy="0 0 0"/>
     <geometry>
-      <mesh filename="file://$(find frame_description)/meshes/holder_4_1.stl" scale="0.001 0.001 0.001"/>
+      <mesh filename="file://$(find drone_frame_description)/meshes/holder_4_1.stl" scale="0.001 0.001 0.001"/>
     </geometry>
     <material name="silver"/>
@@ -220,5 +220,5 @@
     <origin xyz="0.215 -0.02 -0.2" rpy="0 0 0"/>
     <geometry>
-      <mesh filename="file://$(find frame_description)/meshes/holder_4_1.stl" scale="0.001 0.001 0.001"/>
+      <mesh filename="file://$(find drone_frame_description)/meshes/holder_4_1.stl" scale="0.001 0.001 0.001"/>
     </geometry>
   </collision>
@@ -226,12 +226,12 @@
 <link name="holder_3_1">
   <inertial>
-    <origin xyz="0.01627435024563989 3.173676564605099e-10 0.0012743502456399047" rpy="0 0 0"/>
+    <origin xyz="0.016274350245639946 1.6835604438325547e-10 0.0012743502456399047" rpy="0 0 0"/>
     <mass value="0.545696208866394"/>
-    <inertia ixx="0.00016" iyy="0.000161" izz="0.00016" ixy="0.0" iyz="0.0" ixz="1e-06"/>
+    <inertia ixx="0.00016" iyy="0.000161" izz="0.00016" ixy="0.0" iyz="-0.0" ixz="1e-06"/>
   </inertial>
   <visual>
     <origin xyz="0.215 -0.02 0.2" rpy="0 0 0"/>
     <geometry>
-      <mesh filename="file://$(find frame_description)/meshes/holder_3_1.stl" scale="0.001 0.001 0.001"/>
+      <mesh filename="file://$(find drone_frame_description)/meshes/holder_3_1.stl" scale="0.001 0.001 0.001"/>
     </geometry>
     <material name="silver"/>
@@ -240,5 +240,5 @@
     <origin xyz="0.215 -0.02 0.2" rpy="0 0 0"/>
     <geometry>
-      <mesh filename="file://$(find frame_description)/meshes/holder_3_1.stl" scale="0.001 0.001 0.001"/>
+      <mesh filename="file://$(find drone_frame_description)/meshes/holder_3_1.stl" scale="0.001 0.001 0.001"/>
     </geometry>
   </collision>
@@ -246,12 +246,12 @@
 <link name="holder_3_1">
   <inertial>
-    <origin xyz="0.0012743502456399047 3.173676564605099e-10 0.01627435024563989" rpy="0 0 0"/>
+    <origin xyz="0.0012743502456399602 1.6835604438325547e-10 0.01627435024563989" rpy="0 0 0"/>
     <mass value="0.545696208866394"/>
-    <inertia ixx="0.00016" iyy="0.000161" izz="0.00016" ixy="0.0" iyz="0.0" ixz="1e-06"/>
+    <inertia ixx="0.00016" iyy="0.000161" izz="0.00016" ixy="0.0" iyz="-0.0" ixz="1e-06"/>
   </inertial>
   <visual>
     <origin xyz="0.2 -0.02 0.215" rpy="0 0 0"/>
     <geometry>
-      <mesh filename="file://$(find frame_description)/meshes/holder_3_1.stl" scale="0.001 0.001 0.001"/>
+      <mesh filename="file://$(find drone_frame_description)/meshes/holder_3_1.stl" scale="0.001 0.001 0.001"/>
     </geometry>
     <material name="silver"/>
@@ -260,5 +260,5 @@
     <origin xyz="0.2 -0.02 0.215" rpy="0 0 0"/>
     <geometry>
-      <mesh filename="file://$(find frame_description)/meshes/holder_3_1.stl" scale="0.001 0.001 0.001"/>
+      <mesh filename="file://$(find drone_frame_description)/meshes/holder_3_1.stl" scale="0.001 0.001 0.001"/>
     </geometry>
   </collision>
@@ -266,12 +266,12 @@
 <link name="holder_2_1">
   <inertial>
-    <origin xyz="-0.0012743502456399047 -1.9344432306001025e-11 0.01627435024563989" rpy="0 0 0"/>
+    <origin xyz="-0.0012743502456399047 -1.6835604785270242e-10 0.016274350245639946" rpy="0 0 0"/>
     <mass value="0.545696208866394"/>
-    <inertia ixx="0.00016" iyy="0.000161" izz="0.00016" ixy="0.0" iyz="-0.0" ixz="-1e-06"/>
+    <inertia ixx="0.00016" iyy="0.000161" izz="0.00016" ixy="0.0" iyz="0.0" ixz="-1e-06"/>
   </inertial>
   <visual>
     <origin xyz="-0.2 -0.02 0.215" rpy="0 0 0"/>
     <geometry>
-      <mesh filename="file://$(find frame_description)/meshes/holder_2_1.stl" scale="0.001 0.001 0.001"/>
+      <mesh filename="file://$(find drone_frame_description)/meshes/holder_2_1.stl" scale="0.001 0.001 0.001"/>
     </geometry>
     <material name="silver"/>
@@ -280,5 +280,5 @@
     <origin xyz="-0.2 -0.02 0.215" rpy="0 0 0"/>
     <geometry>
-      <mesh filename="file://$(find frame_description)/meshes/holder_2_1.stl" scale="0.001 0.001 0.001"/>
+      <mesh filename="file://$(find drone_frame_description)/meshes/holder_2_1.stl" scale="0.001 0.001 0.001"/>
     </geometry>
   </collision>
@@ -286,12 +286,12 @@
 <link name="holder_2_1">
   <inertial>
-    <origin xyz="-0.01627435024563989 -1.9344432306001025e-11 0.0012743502456399047" rpy="0 0 0"/>
+    <origin xyz="-0.01627435024563989 -1.6835604785270242e-10 0.0012743502456399602" rpy="0 0 0"/>
     <mass value="0.545696208866394"/>
-    <inertia ixx="0.00016" iyy="0.000161" izz="0.00016" ixy="0.0" iyz="-0.0" ixz="-1e-06"/>
+    <inertia ixx="0.00016" iyy="0.000161" izz="0.00016" ixy="0.0" iyz="0.0" ixz="-1e-06"/>
   </inertial>
   <visual>
     <origin xyz="-0.215 -0.02 0.2" rpy="0 0 0"/>
     <geometry>
-      <mesh filename="file://$(find frame_description)/meshes/holder_2_1.stl" scale="0.001 0.001 0.001"/>
+      <mesh filename="file://$(find drone_frame_description)/meshes/holder_2_1.stl" scale="0.001 0.001 0.001"/>
     </geometry>
     <material name="silver"/>
@@ -300,5 +300,5 @@
     <origin xyz="-0.215 -0.02 0.2" rpy="0 0 0"/>
     <geometry>
-      <mesh filename="file://$(find frame_description)/meshes/holder_2_1.stl" scale="0.001 0.001 0.001"/>
+      <mesh filename="file://$(find drone_frame_description)/meshes/holder_2_1.stl" scale="0.001 0.001 0.001"/>
     </geometry>
   </collision>
@@ -313,5 +313,5 @@
     <origin xyz="-0.215 -0.02 -0.2" rpy="0 0 0"/>
     <geometry>
-      <mesh filename="file://$(find frame_description)/meshes/holder_1_1.stl" scale="0.001 0.001 0.001"/>
+      <mesh filename="file://$(find drone_frame_description)/meshes/holder_1_1.stl" scale="0.001 0.001 0.001"/>
     </geometry>
     <material name="silver"/>
@@ -320,5 +320,5 @@
     <origin xyz="-0.215 -0.02 -0.2" rpy="0 0 0"/>
     <geometry>
-      <mesh filename="file://$(find frame_description)/meshes/holder_1_1.stl" scale="0.001 0.001 0.001"/>
+      <mesh filename="file://$(find drone_frame_description)/meshes/holder_1_1.stl" scale="0.001 0.001 0.001"/>
     </geometry>
   </collision>
@@ -333,5 +333,5 @@
     <origin xyz="-0.2 -0.02 -0.215" rpy="0 0 0"/>
     <geometry>
-      <mesh filename="file://$(find frame_description)/meshes/holder_1_1.stl" scale="0.001 0.001 0.001"/>
+      <mesh filename="file://$(find drone_frame_description)/meshes/holder_1_1.stl" scale="0.001 0.001 0.001"/>
     </geometry>
     <material name="silver"/>
@@ -340,5 +340,5 @@
     <origin xyz="-0.2 -0.02 -0.215" rpy="0 0 0"/>
     <geometry>
-      <mesh filename="file://$(find frame_description)/meshes/holder_1_1.stl" scale="0.001 0.001 0.001"/>
+      <mesh filename="file://$(find drone_frame_description)/meshes/holder_1_1.stl" scale="0.001 0.001 0.001"/>
     </geometry>
   </collision>
@@ -353,5 +353,5 @@
     <origin xyz="-0.2 -0.04 -0.2" rpy="0 0 0"/>
     <geometry>
-      <mesh filename="file://$(find frame_description)/meshes/bldc_8_1.stl" scale="0.001 0.001 0.001"/>
+      <mesh filename="file://$(find drone_frame_description)/meshes/bldc_8_1.stl" scale="0.001 0.001 0.001"/>
     </geometry>
     <material name="silver"/>
@@ -360,5 +360,5 @@
     <origin xyz="-0.2 -0.04 -0.2" rpy="0 0 0"/>
     <geometry>
-      <mesh filename="file://$(find frame_description)/meshes/bldc_8_1.stl" scale="0.001 0.001 0.001"/>
+      <mesh filename="file://$(find drone_frame_description)/meshes/bldc_8_1.stl" scale="0.001 0.001 0.001"/>
     </geometry>
   </collision>
@@ -366,5 +366,5 @@
 <link name="bldc_7_1">
   <inertial>
-    <origin xyz="2.6989159021245657e-05 0.012072048037909955 9.851740487398786e-06" rpy="0 0 0"/>
+    <origin xyz="2.6989477628441838e-05 0.012072047888532327 9.8520590945117e-06" rpy="0 0 0"/>
     <mass value="0.22635455509580502"/>
     <inertia ixx="6.6e-05" iyy="0.000112" izz="6.6e-05" ixy="-0.0" iyz="-0.0" ixz="-0.0"/>
@@ -373,5 +373,5 @@
     <origin xyz="-0.2 -0.04 0.2" rpy="0 0 0"/>
     <geometry>
-      <mesh filename="file://$(find frame_description)/meshes/bldc_7_1.stl" scale="0.001 0.001 0.001"/>
+      <mesh filename="file://$(find drone_frame_description)/meshes/bldc_7_1.stl" scale="0.001 0.001 0.001"/>
     </geometry>
     <material name="silver"/>
@@ -380,5 +380,5 @@
     <origin xyz="-0.2 -0.04 0.2" rpy="0 0 0"/>
     <geometry>
-      <mesh filename="file://$(find frame_description)/meshes/bldc_7_1.stl" scale="0.001 0.001 0.001"/>
+      <mesh filename="file://$(find drone_frame_description)/meshes/bldc_7_1.stl" scale="0.001 0.001 0.001"/>
     </geometry>
   </collision>
@@ -386,5 +386,5 @@
 <link name="bldc_6_1">
   <inertial>
-    <origin xyz="2.6989159021273412e-05 0.012072048335933179 9.851740487398786e-06" rpy="0 0 0"/>
+    <origin xyz="2.6989477628469594e-05 0.01207204818675131 9.851421880202604e-06" rpy="0 0 0"/>
     <mass value="0.22635455509580502"/>
     <inertia ixx="6.6e-05" iyy="0.000112" izz="6.6e-05" ixy="-0.0" iyz="-0.0" ixz="-0.0"/>
@@ -393,5 +393,5 @@
     <origin xyz="0.2 -0.04 0.2" rpy="0 0 0"/>
     <geometry>
-      <mesh filename="file://$(find frame_description)/meshes/bldc_6_1.stl" scale="0.001 0.001 0.001"/>
+      <mesh filename="file://$(find drone_frame_description)/meshes/bldc_6_1.stl" scale="0.001 0.001 0.001"/>
     </geometry>
     <material name="silver"/>
@@ -400,5 +400,5 @@
     <origin xyz="0.2 -0.04 0.2" rpy="0 0 0"/>
     <geometry>
-      <mesh filename="file://$(find frame_description)/meshes/bldc_6_1.stl" scale="0.001 0.001 0.001"/>
+      <mesh filename="file://$(find drone_frame_description)/meshes/bldc_6_1.stl" scale="0.001 0.001 0.001"/>
     </geometry>
   </collision>
@@ -406,5 +406,5 @@
 <link name="bldc_5_1">
   <inertial>
-    <origin xyz="-2.6989159019580322e-05 0.01207204803791747 -9.851740487953897e-06" rpy="0 0 0"/>
+    <origin xyz="-2.698947762899695e-05 0.012072047888536115 -9.852059102616328e-06" rpy="0 0 0"/>
     <mass value="0.22635455509580502"/>
     <inertia ixx="6.6e-05" iyy="0.000112" izz="6.6e-05" ixy="0.0" iyz="0.0" ixz="-0.0"/>
@@ -413,5 +413,5 @@
     <origin xyz="0.2 -0.04 -0.2" rpy="0 0 0"/>
     <geometry>
-      <mesh filename="file://$(find frame_description)/meshes/bldc_5_1.stl" scale="0.001 0.001 0.001"/>
+      <mesh filename="file://$(find drone_frame_description)/meshes/bldc_5_1.stl" scale="0.001 0.001 0.001"/>
     </geometry>
     <material name="silver"/>
@@ -420,5 +420,5 @@
     <origin xyz="0.2 -0.04 -0.2" rpy="0 0 0"/>
     <geometry>
-      <mesh filename="file://$(find frame_description)/meshes/bldc_5_1.stl" scale="0.001 0.001 0.001"/>
+      <mesh filename="file://$(find drone_frame_description)/meshes/bldc_5_1.stl" scale="0.001 0.001 0.001"/>
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