Commit message: changed the propeller holder joints

File: urdf/drone_frame.xacro (robot description, xacro)
@@ -146,5 +146,5 @@
 <link name="arm_2_1">
   <inertial>
-    <origin xyz="-0.09732998253804709 -2.5269421971563233e-11 0.08302889455496792" rpy="0 0 0"/>
+    <origin xyz="-0.09732998253804703 -2.5274383280704527e-11 0.08302889455496801" rpy="0 0 0"/>
     <mass value="0.15422742956922936"/>
     <inertia ixx="0.0006" iyy="0.000929" izz="0.000389" ixy="-0.0" iyz="0.0" ixz="0.000277"/>
@@ -186,7 +186,7 @@
 <link name="holder_4_1">
   <inertial>
-    <origin xyz="0.0012743502456467604 -1.6835240493340287e-10 -0.0162743502456395" rpy="0 0 0"/>
+    <origin xyz="0.0012743502456399602 -1.933707013956898e-11 -0.016274350245639946" rpy="0 0 0"/>
     <mass value="0.545696208866394"/>
-    <inertia ixx="0.00016" iyy="0.000161" izz="0.00016" ixy="-0.0" iyz="-0.0" ixz="-1e-06"/>
+    <inertia ixx="0.00016" iyy="0.000161" izz="0.00016" ixy="-0.0" iyz="0.0" ixz="-1e-06"/>
   </inertial>
   <visual>
@@ -206,7 +206,7 @@
 <link name="holder_4_1">
   <inertial>
-    <origin xyz="0.016274350245646746 -1.6835240493340287e-10 -0.0012743502456395162" rpy="0 0 0"/>
+    <origin xyz="0.016274350245639946 -1.933707013956898e-11 -0.0012743502456399602" rpy="0 0 0"/>
     <mass value="0.545696208866394"/>
-    <inertia ixx="0.00016" iyy="0.000161" izz="0.00016" ixy="-0.0" iyz="-0.0" ixz="-1e-06"/>
+    <inertia ixx="0.00016" iyy="0.000161" izz="0.00016" ixy="-0.0" iyz="0.0" ixz="-1e-06"/>
   </inertial>
   <visual>
@@ -226,7 +226,7 @@
 <link name="holder_3_1">
   <inertial>
-    <origin xyz="0.016274350245639946 1.6835604438325547e-10 0.0012743502456399047" rpy="0 0 0"/>
+    <origin xyz="0.01627435024563989 3.173676564605099e-10 0.0012743502456399047" rpy="0 0 0"/>
     <mass value="0.545696208866394"/>
-    <inertia ixx="0.00016" iyy="0.000161" izz="0.00016" ixy="0.0" iyz="-0.0" ixz="1e-06"/>
+    <inertia ixx="0.00016" iyy="0.000161" izz="0.00016" ixy="0.0" iyz="0.0" ixz="1e-06"/>
   </inertial>
   <visual>
@@ -246,7 +246,7 @@
 <link name="holder_3_1">
   <inertial>
-    <origin xyz="0.0012743502456399602 1.6835604438325547e-10 0.01627435024563989" rpy="0 0 0"/>
+    <origin xyz="0.0012743502456399047 3.173676564605099e-10 0.01627435024563989" rpy="0 0 0"/>
     <mass value="0.545696208866394"/>
-    <inertia ixx="0.00016" iyy="0.000161" izz="0.00016" ixy="0.0" iyz="-0.0" ixz="1e-06"/>
+    <inertia ixx="0.00016" iyy="0.000161" izz="0.00016" ixy="0.0" iyz="0.0" ixz="1e-06"/>
   </inertial>
   <visual>
@@ -266,7 +266,7 @@
 <link name="holder_2_1">
   <inertial>
-    <origin xyz="-0.0012743502456399047 -1.6835604785270242e-10 0.016274350245639946" rpy="0 0 0"/>
+    <origin xyz="-0.0012743502456399047 -1.9344432306001025e-11 0.01627435024563989" rpy="0 0 0"/>
     <mass value="0.545696208866394"/>
-    <inertia ixx="0.00016" iyy="0.000161" izz="0.00016" ixy="0.0" iyz="0.0" ixz="-1e-06"/>
+    <inertia ixx="0.00016" iyy="0.000161" izz="0.00016" ixy="0.0" iyz="-0.0" ixz="-1e-06"/>
   </inertial>
   <visual>
@@ -286,7 +286,7 @@
 <link name="holder_2_1">
   <inertial>
-    <origin xyz="-0.01627435024563989 -1.6835604785270242e-10 0.0012743502456399602" rpy="0 0 0"/>
+    <origin xyz="-0.01627435024563989 -1.9344432306001025e-11 0.0012743502456399047" rpy="0 0 0"/>
     <mass value="0.545696208866394"/>
-    <inertia ixx="0.00016" iyy="0.000161" izz="0.00016" ixy="0.0" iyz="0.0" ixz="-1e-06"/>
+    <inertia ixx="0.00016" iyy="0.000161" izz="0.00016" ixy="0.0" iyz="-0.0" ixz="-1e-06"/>
   </inertial>
   <visual>
@@ -366,5 +366,5 @@
 <link name="bldc_7_1">
   <inertial>
-    <origin xyz="2.6989477628441838e-05 0.012072047888532327 9.8520590945117e-06" rpy="0 0 0"/>
+    <origin xyz="2.6989159021245657e-05 0.012072048037909955 9.851740487398786e-06" rpy="0 0 0"/>
     <mass value="0.22635455509580502"/>
     <inertia ixx="6.6e-05" iyy="0.000112" izz="6.6e-05" ixy="-0.0" iyz="-0.0" ixz="-0.0"/>
@@ -386,5 +386,5 @@
 <link name="bldc_6_1">
   <inertial>
-    <origin xyz="2.6989477628469594e-05 0.01207204818675131 9.851421880202604e-06" rpy="0 0 0"/>
+    <origin xyz="2.6989159021273412e-05 0.012072048335933179 9.851740487398786e-06" rpy="0 0 0"/>
     <mass value="0.22635455509580502"/>
     <inertia ixx="6.6e-05" iyy="0.000112" izz="6.6e-05" ixy="-0.0" iyz="-0.0" ixz="-0.0"/>
@@ -406,5 +406,5 @@
 <link name="bldc_5_1">
   <inertial>
-    <origin xyz="-2.698947762899695e-05 0.012072047888536115 -9.852059102616328e-06" rpy="0 0 0"/>
+    <origin xyz="-2.6989159019580322e-05 0.01207204803791747 -9.851740487953897e-06" rpy="0 0 0"/>
     <mass value="0.22635455509580502"/>
     <inertia ixx="6.6e-05" iyy="0.000112" izz="6.6e-05" ixy="0.0" iyz="0.0" ixz="-0.0"/>
@@ -426,10 +426,10 @@
 <link name="bldc_4_1">
   <inertial>
-    <origin xyz="-2.6989477628414082e-05 -0.012072048186751306 9.851421880202604e-06" rpy="0 0 0"/>
+    <origin xyz="-2.6989159021273412e-05 -0.012072048037909955 9.851740487398786e-06" rpy="0 0 0"/>
     <mass value="0.22635455509580502"/>
     <inertia ixx="6.6e-05" iyy="0.000112" izz="6.6e-05" ixy="-0.0" iyz="0.0" ixz="0.0"/>
   </inertial>
   <visual>
-    <origin xyz="-0.2 0.0 0.2" rpy="0 0 0"/>
+    <origin xyz="-0.2 -0.0 0.2" rpy="0 0 0"/>
     <geometry>
       <mesh filename="file://$(find drone_frame_description)/meshes/bldc_4_1.stl" scale="0.001 0.001 0.001"/>
@@ -438,5 +438,5 @@
   </visual>
   <collision>
-    <origin xyz="-0.2 0.0 0.2" rpy="0 0 0"/>
+    <origin xyz="-0.2 -0.0 0.2" rpy="0 0 0"/>
     <geometry>
       <mesh filename="file://$(find drone_frame_description)/meshes/bldc_4_1.stl" scale="0.001 0.001 0.001"/>
@@ -446,5 +446,5 @@
 <link name="bldc_3_1">
   <inertial>
-    <origin xyz="-2.6989477628414082e-05 -0.012072047888532344 9.8520590945117e-06" rpy="0 0 0"/>
+    <origin xyz="-2.6989159021245657e-05 -0.01207204773988673 9.851740487398786e-06" rpy="0 0 0"/>
     <mass value="0.22635455509580502"/>
     <inertia ixx="6.6e-05" iyy="0.000112" izz="6.6e-05" ixy="-0.0" iyz="0.0" ixz="0.0"/>
@@ -466,10 +466,10 @@
 <link name="bldc_2_1">
   <inertial>
-    <origin xyz="2.698947764109838e-05 -0.012072048186747673 -9.85142187226451e-06" rpy="0 0 0"/>
+    <origin xyz="2.6989159019635833e-05 -0.012072048037902619 -9.851740487953897e-06" rpy="0 0 0"/>
     <mass value="0.22635455509580502"/>
     <inertia ixx="6.6e-05" iyy="0.000112" izz="6.6e-05" ixy="0.0" iyz="-0.0" ixz="0.0"/>
   </inertial>
   <visual>
-    <origin xyz="0.2 0.0 -0.2" rpy="0 0 0"/>
+    <origin xyz="0.2 -0.0 -0.2" rpy="0 0 0"/>
     <geometry>
       <mesh filename="file://$(find drone_frame_description)/meshes/bldc_2_1.stl" scale="0.001 0.001 0.001"/>
@@ -478,5 +478,5 @@
   </visual>
   <collision>
-    <origin xyz="0.2 0.0 -0.2" rpy="0 0 0"/>
+    <origin xyz="0.2 -0.0 -0.2" rpy="0 0 0"/>
     <geometry>
       <mesh filename="file://$(find drone_frame_description)/meshes/bldc_2_1.stl" scale="0.001 0.001 0.001"/>
@@ -606,7 +606,7 @@
 <link name="prop_7_1">
   <inertial>
-    <origin xyz="5.247765000326865e-10 0.0014016425752792078 5.1846385240583714e-09" rpy="0 0 0"/>
+    <origin xyz="9.956764301932708e-10 0.001401642724294494 5.655541951421483e-09" rpy="0 0 0"/>
     <mass value="0.0335765475239113"/>
-    <inertia ixx="0.00011" iyy="0.000111" izz="1e-06" ixy="0.0" iyz="-0.0" ixz="-1e-06"/>
+    <inertia ixx="0.00011" iyy="0.000111" izz="1e-06" ixy="0.0" iyz="0.0" ixz="-1e-06"/>
   </inertial>
   <visual>
@@ -626,5 +626,5 @@
 <link name="prop_6_1">
   <inertial>
-    <origin xyz="-5.247808854136338e-10 0.0014016428732985392 -6.126436385978096e-09" rpy="0 0 0"/>
+    <origin xyz="-9.956739044358898e-10 0.0014016430223102033 -5.65554336695584e-09" rpy="0 0 0"/>
     <mass value="0.0335765475239113"/>
     <inertia ixx="0.00011" iyy="0.000111" izz="1e-06" ixy="-0.0" iyz="-0.0" ixz="-1e-06"/>
@@ -646,7 +646,7 @@
 <link name="prop_5_1">
   <inertial>
-    <origin xyz="-5.247809131692094e-10 0.0014016425752753914 -5.184650347933584e-09" rpy="0 0 0"/>
+    <origin xyz="-9.956739321914654e-10 0.001401642724286986 -5.655543339200264e-09" rpy="0 0 0"/>
     <mass value="0.0335765475239113"/>
-    <inertia ixx="0.00011" iyy="0.000111" izz="1e-06" ixy="-0.0" iyz="0.0" ixz="-1e-06"/>
+    <inertia ixx="0.00011" iyy="0.000111" izz="1e-06" ixy="-0.0" iyz="-0.0" ixz="-1e-06"/>
   </inertial>
   <visual>
@@ -840,51 +840,59 @@
   <limit upper="1.570796" lower="-1.570796" effort="100" velocity="100"/>
 </joint>
-<joint name="Revolute 13" type="continuous">
+<joint name="Revolute 13" type="revolute">
   <origin xyz="-0.16 0.0 0.0" rpy="0 0 0"/>
   <parent link="arm_1_1"/>
   <child link="holder_4_1"/>
   <axis xyz="-0.0 0.0 -1.0"/>
-</joint>
-<joint name="Revolute 14" type="continuous">
+  <limit upper="1.570796" lower="-1.570796" effort="100" velocity="100"/>
+</joint>
+<joint name="Revolute 14" type="revolute">
   <origin xyz="-0.015 0.0 0.145" rpy="0 0 0"/>
   <parent link="arm_2_1"/>
   <child link="holder_4_1"/>
-  <axis xyz="1.0 -0.0 -0.0"/>
-</joint>
-<joint name="Revolute 15" type="continuous">
+  <axis xyz="1.0 0.0 -0.0"/>
+  <limit upper="1.570796" lower="-1.570796" effort="100" velocity="100"/>
+</joint>
+<joint name="Revolute 15" type="revolute">
   <origin xyz="0.0 0.0 -0.16" rpy="0 0 0"/>
   <parent link="arm_8_1"/>
   <child link="holder_3_1"/>
   <axis xyz="1.0 0.0 0.0"/>
-</joint>
-<joint name="Revolute 16" type="continuous">
+  <limit upper="1.570796" lower="-1.570796" effort="100" velocity="100"/>
+</joint>
+<joint name="Revolute 16" type="revolute">
   <origin xyz="-0.145 0.0 -0.015" rpy="0 0 0"/>
   <parent link="arm_7_1"/>
   <child link="holder_3_1"/>
   <axis xyz="0.0 0.0 1.0"/>
-</joint>
-<joint name="Revolute 17" type="continuous">
+  <limit upper="1.570796" lower="-1.570796" effort="100" velocity="100"/>
+</joint>
+<joint name="Revolute 17" type="revolute">
   <origin xyz="0.16 0.0 0.0" rpy="0 0 0"/>
   <parent link="arm_3_1"/>
   <child link="holder_2_1"/>
   <axis xyz="0.0 0.0 1.0"/>
-</joint>
-<joint name="Revolute 18" type="continuous">
+  <limit upper="1.570796" lower="-1.570796" effort="100" velocity="100"/>
+</joint>
+<joint name="Revolute 18" type="revolute">
   <origin xyz="0.015 0.0 -0.145" rpy="0 0 0"/>
   <parent link="arm_4_1"/>
   <child link="holder_2_1"/>
   <axis xyz="-1.0 0.0 0.0"/>
-</joint>
-<joint name="Revolute 19" type="continuous">
+  <limit upper="1.570796" lower="-1.570796" effort="100" velocity="100"/>
+</joint>
+<joint name="Revolute 19" type="revolute">
   <origin xyz="0.0 0.0 0.16" rpy="0 0 0"/>
   <parent link="arm_6_1"/>
   <child link="holder_1_1"/>
   <axis xyz="-1.0 -0.0 -0.0"/>
-</joint>
-<joint name="Revolute 20" type="continuous">
+  <limit upper="1.570796" lower="-1.570796" effort="100" velocity="100"/>
+</joint>
+<joint name="Revolute 20" type="revolute">
   <origin xyz="0.145 0.0 0.015" rpy="0 0 0"/>
   <parent link="arm_5_1"/>
   <child link="holder_1_1"/>
   <axis xyz="0.0 0.0 -1.0"/>
+  <limit upper="1.570796" lower="-1.570796" effort="100" velocity="100"/>
 </joint>
 <joint name="Rigid 21" type="fixed">
@@ -958,5 +966,5 @@
   <parent link="bldc_5_1"/>
   <child link="prop_7_1"/>
-  <axis xyz="0.0 -1.0 0.0"/>
+  <axis xyz="-0.0 -1.0 0.0"/>
 </joint>
 <joint name="Revolute 35" type="continuous">
@@ -964,5 +972,5 @@
   <parent link="bldc_6_1"/>
   <child link="prop_6_1"/>
-  <axis xyz="-0.0 -1.0 0.0"/>
+  <axis xyz="0.0 -1.0 -0.0"/>
 </joint>
 <joint name="Revolute 36" type="continuous">
@@ -970,5 +978,5 @@
   <parent link="bldc_7_1"/>
   <child link="prop_5_1"/>
-  <axis xyz="-0.0 -1.0 -0.0"/>
+  <axis xyz="0.0 -1.0 -0.0"/>
 </joint>
 <joint name="Revolute 37" type="continuous">
@@ -976,5 +984,5 @@
   <parent link="bldc_4_1"/>
   <child link="prop_4_1"/>
-  <axis xyz="0.0 1.0 0.0"/>
+  <axis xyz="-0.0 1.0 -0.0"/>
 </joint>
 <joint name="Revolute 38" type="continuous">
@@ -988,5 +996,5 @@
   <parent link="bldc_3_1"/>
   <child link="prop_2_1"/>
-  <axis xyz="0.0 1.0 -0.0"/>
+  <axis xyz="-0.0 1.0 -0.0"/>
 </joint>
 <joint name="Revolute 40" type="continuous">
@@ -994,5 +1002,5 @@
   <parent link="bldc_2_1"/>
   <child link="prop_1_1"/>
-  <axis xyz="-0.0 1.0 -0.0"/>
+  <axis xyz="0.0 1.0 0.0"/>
 </joint>
 <joint name="Rigid 41" type="fixed">
