Commit message: fixed the bridging error

File: drone_frame_description/urdf/coaxial_holder.xacro (robot description, xacro)
@@ -5,5 +5,5 @@
     <inertial>
       <origin xyz="${io}" rpy="0 0 0"/>
-      <mass value="0.545696208866394"/>
+      <mass value="0.3"/>
       <inertia ixx="${ixx}" iyy="${iyy}" izz="${izz}" ixy="${ixy}" iyz="${iyz}" ixz="${ixz}"/>
     </inertial>
@@ -47,5 +47,5 @@
     <inertial>
       <origin xyz="${io}" rpy="0 0 0"/>
-      <mass value="0.22635455509580407"/>
+      <mass value="0.25"/>
       <inertia ixx="6.6e-05" iyy="0.000112" izz="6.6e-05" ixy="${ixy}" iyz="${iyz}" ixz="${ixz}"/>
     </inertial>

File: drone_frame_description/urdf/thruster.xacro (robot description, xacro)
@@ -53,11 +53,11 @@
       <joint_name>thruster_joint_${prop_num}</joint_name>
       <topic>thruster_${prop_num}/cmd</topic>
-      <thrust_coefficient>0.015</thrust_coefficient>
+      <thrust_coefficient>0.125</thrust_coefficient>
       <fluid_density>1.225</fluid_density>
       <propeller_diameter>0.2286</propeller_diameter>
       <velocity_control>true</velocity_control>
       <use_angvel_cmd>false</use_angvel_cmd>
-      <max_thrust_cmd>40</max_thrust_cmd>
-      <min_thrust_cmd>-40</min_thrust_cmd>
+      <max_thrust_cmd>200</max_thrust_cmd>
+      <min_thrust_cmd>-200</min_thrust_cmd>
       <direction>${direction}</direction>
     </plugin>
