Commit message: changed xacro files

File: drone_frame_description/urdf/drone_frame.xacro (robot description, xacro)
@@ -24,405 +24,5 @@
   </collision>
 </link>
-<link name="arm_8_1">
-  <inertial>
-    <origin xyz="-0.0973299825380552 2.527436940291672e-11 -0.08302889455495804" rpy="0 0 0"/>
-    <mass value="0.15422742956922936"/>
-    <inertia ixx="0.0006" iyy="0.000929" izz="0.000389" ixy="0.0" iyz="0.0" ixz="-0.000277"/>
-  </inertial>
-  <visual>
-    <origin xyz="0.2 -0.02 0.055" rpy="0 0 0"/>
-    <geometry>
-      <mesh filename="file://$(find drone_frame_description)/meshes/arm_8_1.stl" scale="0.001 0.001 0.001"/>
-    </geometry>
-    <material name="black"/>
-  </visual>
-  <collision>
-    <origin xyz="0.2 -0.02 0.055" rpy="0 0 0"/>
-    <geometry>
-      <mesh filename="file://$(find drone_frame_description)/meshes/arm_8_1.stl" scale="0.001 0.001 0.001"/>
-    </geometry>
-  </collision>
-</link>
-<link name="arm_7_1">
-  <inertial>
-    <origin xyz="-0.08302889455495802 -2.527437287236367e-11 -0.0973299825380552" rpy="0 0 0"/>
-    <mass value="0.15422742956922936"/>
-    <inertia ixx="0.000389" iyy="0.000929" izz="0.0006" ixy="-0.0" iyz="-0.0" ixz="-0.000277"/>
-  </inertial>
-  <visual>
-    <origin xyz="0.055 -0.02 0.2" rpy="0 0 0"/>
-    <geometry>
-      <mesh filename="file://$(find drone_frame_description)/meshes/arm_7_1.stl" scale="0.001 0.001 0.001"/>
-    </geometry>
-    <material name="black"/>
-  </visual>
-  <collision>
-    <origin xyz="0.055 -0.02 0.2" rpy="0 0 0"/>
-    <geometry>
-      <mesh filename="file://$(find drone_frame_description)/meshes/arm_7_1.stl" scale="0.001 0.001 0.001"/>
-    </geometry>
-  </collision>
-</link>
-<link name="arm_6_1">
-  <inertial>
-    <origin xyz="0.09732998253805486 2.5274376341810623e-11 0.08302889455495802" rpy="0 0 0"/>
-    <mass value="0.15422742956922936"/>
-    <inertia ixx="0.0006" iyy="0.000929" izz="0.000389" ixy="-0.0" iyz="-0.0" ixz="-0.000277"/>
-  </inertial>
-  <visual>
-    <origin xyz="-0.2 -0.02 -0.055" rpy="0 0 0"/>
-    <geometry>
-      <mesh filename="file://$(find drone_frame_description)/meshes/arm_6_1.stl" scale="0.001 0.001 0.001"/>
-    </geometry>
-    <material name="black"/>
-  </visual>
-  <collision>
-    <origin xyz="-0.2 -0.02 -0.055" rpy="0 0 0"/>
-    <geometry>
-      <mesh filename="file://$(find drone_frame_description)/meshes/arm_6_1.stl" scale="0.001 0.001 0.001"/>
-    </geometry>
-  </collision>
-</link>
-<link name="arm_5_1">
-  <inertial>
-    <origin xyz="0.08302889455495802 -2.527437287236367e-11 0.0973299825380552" rpy="0 0 0"/>
-    <mass value="0.15422742956922936"/>
-    <inertia ixx="0.000389" iyy="0.000929" izz="0.0006" ixy="0.0" iyz="0.0" ixz="-0.000277"/>
-  </inertial>
-  <visual>
-    <origin xyz="-0.055 -0.02 -0.2" rpy="0 0 0"/>
-    <geometry>
-      <mesh filename="file://$(find drone_frame_description)/meshes/arm_5_1.stl" scale="0.001 0.001 0.001"/>
-    </geometry>
-    <material name="black"/>
-  </visual>
-  <collision>
-    <origin xyz="-0.055 -0.02 -0.2" rpy="0 0 0"/>
-    <geometry>
-      <mesh filename="file://$(find drone_frame_description)/meshes/arm_5_1.stl" scale="0.001 0.001 0.001"/>
-    </geometry>
-  </collision>
-</link>
-<link name="arm_4_1">
-  <inertial>
-    <origin xyz="0.0973299825380552 -2.527437287236367e-11 -0.08302889455495804" rpy="0 0 0"/>
-    <mass value="0.15422742956922936"/>
-    <inertia ixx="0.0006" iyy="0.000929" izz="0.000389" ixy="0.0" iyz="-0.0" ixz="0.000277"/>
-  </inertial>
-  <visual>
-    <origin xyz="-0.2 -0.02 0.055" rpy="0 0 0"/>
-    <geometry>
-      <mesh filename="file://$(find drone_frame_description)/meshes/arm_4_1.stl" scale="0.001 0.001 0.001"/>
-    </geometry>
-    <material name="black"/>
-  </visual>
-  <collision>
-    <origin xyz="-0.2 -0.02 0.055" rpy="0 0 0"/>
-    <geometry>
-      <mesh filename="file://$(find drone_frame_description)/meshes/arm_4_1.stl" scale="0.001 0.001 0.001"/>
-    </geometry>
-  </collision>
-</link>
-<link name="arm_3_1">
-  <inertial>
-    <origin xyz="0.08302889455495802 2.527436940291672e-11 -0.0973299825380552" rpy="0 0 0"/>
-    <mass value="0.15422742956922936"/>
-    <inertia ixx="0.000389" iyy="0.000929" izz="0.0006" ixy="-0.0" iyz="0.0" ixz="0.000277"/>
-  </inertial>
-  <visual>
-    <origin xyz="-0.055 -0.02 0.2" rpy="0 0 0"/>
-    <geometry>
-      <mesh filename="file://$(find drone_frame_description)/meshes/arm_3_1.stl" scale="0.001 0.001 0.001"/>
-    </geometry>
-    <material name="black"/>
-  </visual>
-  <collision>
-    <origin xyz="-0.055 -0.02 0.2" rpy="0 0 0"/>
-    <geometry>
-      <mesh filename="file://$(find drone_frame_description)/meshes/arm_3_1.stl" scale="0.001 0.001 0.001"/>
-    </geometry>
-  </collision>
-</link>
-<link name="arm_2_1">
-  <inertial>
-    <origin xyz="-0.09732998253804703 -2.5274383280704527e-11 0.08302889455496801" rpy="0 0 0"/>
-    <mass value="0.15422742956922936"/>
-    <inertia ixx="0.0006" iyy="0.000929" izz="0.000389" ixy="-0.0" iyz="0.0" ixz="0.000277"/>
-  </inertial>
-  <visual>
-    <origin xyz="0.2 -0.02 -0.055" rpy="0 0 0"/>
-    <geometry>
-      <mesh filename="file://$(find drone_frame_description)/meshes/arm_2_1.stl" scale="0.001 0.001 0.001"/>
-    </geometry>
-    <material name="black"/>
-  </visual>
-  <collision>
-    <origin xyz="0.2 -0.02 -0.055" rpy="0 0 0"/>
-    <geometry>
-      <mesh filename="file://$(find drone_frame_description)/meshes/arm_2_1.stl" scale="0.001 0.001 0.001"/>
-    </geometry>
-  </collision>
-</link>
-<link name="arm_1_1">
-  <inertial>
-    <origin xyz="-0.08302889455495796 2.5278622944879814e-11 0.0973299825380552" rpy="0 0 0"/>
-    <mass value="0.15422742956922936"/>
-    <inertia ixx="0.000389" iyy="0.000929" izz="0.0006" ixy="0.0" iyz="-0.0" ixz="0.000277"/>
-  </inertial>
-  <visual>
-    <origin xyz="0.055 -0.02 -0.2" rpy="0 0 0"/>
-    <geometry>
-      <mesh filename="file://$(find drone_frame_description)/meshes/arm_1_1.stl" scale="0.001 0.001 0.001"/>
-    </geometry>
-    <material name="black"/>
-  </visual>
-  <collision>
-    <origin xyz="0.055 -0.02 -0.2" rpy="0 0 0"/>
-    <geometry>
-      <mesh filename="file://$(find drone_frame_description)/meshes/arm_1_1.stl" scale="0.001 0.001 0.001"/>
-    </geometry>
-  </collision>
-</link>
-<link name="holder_4">
-  <inertial>
-    <origin xyz="0.0012743502456399602 -1.933707013956898e-11 -0.016274350245639946" rpy="0 0 0"/>
-    <mass value="0.545696208866394"/>
-    <inertia ixx="0.00016" iyy="0.000161" izz="0.00016" ixy="-0.0" iyz="0.0" ixz="-1e-06"/>
-  </inertial>
-  <visual>
-    <origin xyz="0.215 -0.02 -0.2" rpy="0 0 0"/>
-    <geometry>
-      <mesh filename="file://$(find drone_frame_description)/meshes/holder_4_1.stl" scale="0.001 0.001 0.001"/>
-    </geometry>
-    <material name="silver"/>
-  </visual>
-  <collision>
-    <origin xyz="0.2 -0.02 -0.215" rpy="0 0 0"/>
-    <geometry>
-      <mesh filename="file://$(find drone_frame_description)/meshes/holder_4_1.stl" scale="0.001 0.001 0.001"/>
-    </geometry>
-  </collision>
-</link>
-<link name="holder_3">
-  <inertial>
-    <origin xyz="0.01627435024563989 3.173676564605099e-10 0.0012743502456399047" rpy="0 0 0"/>
-    <mass value="0.545696208866394"/>
-    <inertia ixx="0.00016" iyy="0.000161" izz="0.00016" ixy="0.0" iyz="0.0" ixz="1e-06"/>
-  </inertial>
-  <visual>
-    <origin xyz="0.20 -0.02 0.215" rpy="0 0 0"/>
-    <geometry>
-      <mesh filename="file://$(find drone_frame_description)/meshes/holder_3_1.stl" scale="0.001 0.001 0.001"/>
-    </geometry>
-    <material name="silver"/>
-  </visual>
-  <collision>
-    <origin xyz="0.215 -0.02 0.215" rpy="0 0 0"/>
-    <geometry>
-      <mesh filename="file://$(find drone_frame_description)/meshes/holder_3_1.stl" scale="0.001 0.001 0.001"/>
-    </geometry>
-  </collision>
-</link>
-<link name="holder_2">
-  <inertial>
-    <origin xyz="-0.0012743502456399047 -1.9344432306001025e-11 0.01627435024563989" rpy="0 0 0"/>
-    <mass value="0.545696208866394"/>
-    <inertia ixx="0.00016" iyy="0.000161" izz="0.00016" ixy="0.0" iyz="-0.0" ixz="-1e-06"/>
-  </inertial>
-  <visual>
-    <origin xyz="-0.215 -0.02 0.2" rpy="0 0 0"/>
-    <geometry>
-      <mesh filename="file://$(find drone_frame_description)/meshes/holder_2_1.stl" scale="0.001 0.001 0.001"/>
-    </geometry>
-    <material name="silver"/>
-  </visual>
-  <collision>
-    <origin xyz="-0.2 -0.02 0.215" rpy="0 0 0"/>
-    <geometry>
-      <mesh filename="file://$(find drone_frame_description)/meshes/holder_2_1.stl" scale="0.001 0.001 0.001"/>
-    </geometry>
-  </collision>
-</link>
-<link name="holder_1">
-  <inertial>
-    <origin xyz="-0.01627435024563989 -1.9344414958766265e-11 -0.0012743502456399047" rpy="0 0 0"/>
-    <mass value="0.545696208866394"/>
-    <inertia ixx="0.00016" iyy="0.000161" izz="0.00016" ixy="0.0" iyz="0.0" ixz="1e-06"/>
-  </inertial>
-  <visual>
-    <origin xyz="-0.2 -0.02 -0.215" rpy="0 0 0"/>
-    <geometry>
-      <mesh filename="file://$(find drone_frame_description)/meshes/holder_1_1.stl" scale="0.001 0.001 0.001"/>
-    </geometry>
-    <material name="silver"/>
-  </visual>
-  <collision>
-    <origin xyz="-0.215 -0.02 -0.2" rpy="0 0 0"/>
-    <geometry>
-      <mesh filename="file://$(find drone_frame_description)/meshes/holder_1_1.stl" scale="0.001 0.001 0.001"/>
-    </geometry>
-  </collision>
-</link>
-<link name="bldc_8_1">
-  <inertial>
-    <origin xyz="-9.850613495537841e-06 0.012072048037910045 2.6988692206020293e-05" rpy="0 0 0"/>
-    <mass value="0.22635455509580407"/>
-    <inertia ixx="6.6e-05" iyy="0.000112" izz="6.6e-05" ixy="0.0" iyz="-0.0" ixz="0.0"/>
-  </inertial>
-  <visual>
-    <origin xyz="-0.2 -0.04 -0.2" rpy="0 0 0"/>
-    <geometry>
-      <mesh filename="file://$(find drone_frame_description)/meshes/bldc_8_1.stl" scale="0.001 0.001 0.001"/>
-    </geometry>
-    <material name="silver"/>
-  </visual>
-  <collision>
-    <origin xyz="-0.2 -0.04 -0.2" rpy="0 0 0"/>
-    <geometry>
-      <mesh filename="file://$(find drone_frame_description)/meshes/bldc_8_1.stl" scale="0.001 0.001 0.001"/>
-    </geometry>
-  </collision>
-</link>
-<link name="bldc_7_1">
-  <inertial>
-    <origin xyz="2.6989159021245657e-05 0.012072048037909955 9.851740487398786e-06" rpy="0 0 0"/>
-    <mass value="0.22635455509580502"/>
-    <inertia ixx="6.6e-05" iyy="0.000112" izz="6.6e-05" ixy="-0.0" iyz="-0.0" ixz="-0.0"/>
-  </inertial>
-  <visual>
-    <origin xyz="-0.2 -0.04 0.2" rpy="0 0 0"/>
-    <geometry>
-      <mesh filename="file://$(find drone_frame_description)/meshes/bldc_7_1.stl" scale="0.001 0.001 0.001"/>
-    </geometry>
-    <material name="silver"/>
-  </visual>
-  <collision>
-    <origin xyz="-0.2 -0.04 0.2" rpy="0 0 0"/>
-    <geometry>
-      <mesh filename="file://$(find drone_frame_description)/meshes/bldc_7_1.stl" scale="0.001 0.001 0.001"/>
-    </geometry>
-  </collision>
-</link>
-<link name="bldc_6_1">
-  <inertial>
-    <origin xyz="2.6989159021273412e-05 0.012072048335933179 9.851740487398786e-06" rpy="0 0 0"/>
-    <mass value="0.22635455509580502"/>
-    <inertia ixx="6.6e-05" iyy="0.000112" izz="6.6e-05" ixy="-0.0" iyz="-0.0" ixz="-0.0"/>
-  </inertial>
-  <visual>
-    <origin xyz="0.2 -0.04 0.2" rpy="0 0 0"/>
-    <geometry>
-      <mesh filename="file://$(find drone_frame_description)/meshes/bldc_6_1.stl" scale="0.001 0.001 0.001"/>
-    </geometry>
-    <material name="silver"/>
-  </visual>
-  <collision>
-    <origin xyz="0.2 -0.04 0.2" rpy="0 0 0"/>
-    <geometry>
-      <mesh filename="file://$(find drone_frame_description)/meshes/bldc_6_1.stl" scale="0.001 0.001 0.001"/>
-    </geometry>
-  </collision>
-</link>
-<link name="bldc_5_1">
-  <inertial>
-    <origin xyz="-2.6989159019580322e-05 0.01207204803791747 -9.851740487953897e-06" rpy="0 0 0"/>
-    <mass value="0.22635455509580502"/>
-    <inertia ixx="6.6e-05" iyy="0.000112" izz="6.6e-05" ixy="0.0" iyz="0.0" ixz="-0.0"/>
-  </inertial>
-  <visual>
-    <origin xyz="0.2 -0.04 -0.2" rpy="0 0 0"/>
-    <geometry>
-      <mesh filename="file://$(find drone_frame_description)/meshes/bldc_5_1.stl" scale="0.001 0.001 0.001"/>
-    </geometry>
-    <material name="silver"/>
-  </visual>
-  <collision>
-    <origin xyz="0.2 -0.04 -0.2" rpy="0 0 0"/>
-    <geometry>
-      <mesh filename="file://$(find drone_frame_description)/meshes/bldc_5_1.stl" scale="0.001 0.001 0.001"/>
-    </geometry>
-  </collision>
-</link>
-<link name="bldc_4_1">
-  <inertial>
-    <origin xyz="-2.6989159021273412e-05 -0.012072048037909955 9.851740487398786e-06" rpy="0 0 0"/>
-    <mass value="0.22635455509580502"/>
-    <inertia ixx="6.6e-05" iyy="0.000112" izz="6.6e-05" ixy="-0.0" iyz="0.0" ixz="0.0"/>
-  </inertial>
-  <visual>
-    <origin xyz="-0.2 -0.0 0.2" rpy="0 0 0"/>
-    <geometry>
-      <mesh filename="file://$(find drone_frame_description)/meshes/bldc_4_1.stl" scale="0.001 0.001 0.001"/>
-    </geometry>
-    <material name="silver"/>
-  </visual>
-  <collision>
-    <origin xyz="-0.2 -0.0 0.2" rpy="0 0 0"/>
-    <geometry>
-      <mesh filename="file://$(find drone_frame_description)/meshes/bldc_4_1.stl" scale="0.001 0.001 0.001"/>
-    </geometry>
-  </collision>
-</link>
-<link name="bldc_3_1">
-  <inertial>
-    <origin xyz="-2.6989159021245657e-05 -0.01207204773988673 9.851740487398786e-06" rpy="0 0 0"/>
-    <mass value="0.22635455509580502"/>
-    <inertia ixx="6.6e-05" iyy="0.000112" izz="6.6e-05" ixy="-0.0" iyz="0.0" ixz="0.0"/>
-  </inertial>
-  <visual>
-    <origin xyz="0.2 -0.0 0.2" rpy="0 0 0"/>
-    <geometry>
-      <mesh filename="file://$(find drone_frame_description)/meshes/bldc_3_1.stl" scale="0.001 0.001 0.001"/>
-    </geometry>
-    <material name="silver"/>
-  </visual>
-  <collision>
-    <origin xyz="0.2 -0.0 0.2" rpy="0 0 0"/>
-    <geometry>
-      <mesh filename="file://$(find drone_frame_description)/meshes/bldc_3_1.stl" scale="0.001 0.001 0.001"/>
-    </geometry>
-  </collision>
-</link>
-<link name="bldc_2_1">
-  <inertial>
-    <origin xyz="2.6989159019635833e-05 -0.012072048037902619 -9.851740487953897e-06" rpy="0 0 0"/>
-    <mass value="0.22635455509580502"/>
-    <inertia ixx="6.6e-05" iyy="0.000112" izz="6.6e-05" ixy="0.0" iyz="-0.0" ixz="0.0"/>
-  </inertial>
-  <visual>
-    <origin xyz="0.2 -0.0 -0.2" rpy="0 0 0"/>
-    <geometry>
-      <mesh filename="file://$(find drone_frame_description)/meshes/bldc_2_1.stl" scale="0.001 0.001 0.001"/>
-    </geometry>
-    <material name="silver"/>
-  </visual>
-  <collision>
-    <origin xyz="0.2 -0.0 -0.2" rpy="0 0 0"/>
-    <geometry>
-      <mesh filename="file://$(find drone_frame_description)/meshes/bldc_2_1.stl" scale="0.001 0.001 0.001"/>
-    </geometry>
-  </collision>
-</link>
-<link name="bldc_1_1">
-  <inertial>
-    <origin xyz="-9.85174048737103e-06 -0.012072048037909984 -2.6989159021245657e-05" rpy="0 0 0"/>
-    <mass value="0.22635455509580502"/>
-    <inertia ixx="6.6e-05" iyy="0.000112" izz="6.6e-05" ixy="-0.0" iyz="-0.0" ixz="-0.0"/>
-  </inertial>
-  <visual>
-    <origin xyz="-0.2 0.0 -0.2" rpy="0 0 0"/>
-    <geometry>
-      <mesh filename="file://$(find drone_frame_description)/meshes/bldc_1_1.stl" scale="0.001 0.001 0.001"/>
-    </geometry>
-    <material name="silver"/>
-  </visual>
-  <collision>
-    <origin xyz="-0.2 0.0 -0.2" rpy="0 0 0"/>
-    <geometry>
-      <mesh filename="file://$(find drone_frame_description)/meshes/bldc_1_1.stl" scale="0.001 0.001 0.001"/>
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
Commit message: included the world

File: drone_frame_description/urdf/drone_frame.xacro (robot description, xacro)
@@ -23,5 +23,5 @@
   </collision>
 </link>
-<link name="controller">
+<!-- <link name="controller">
   <inertial>
     <origin xyz="0.029999999999999964 0.0075 -0.08999999999999991" rpy="0 0 0"/>
@@ -172,5 +172,5 @@
   <parent link="base_link"/>
   <child link="testing_probe"/>
-</joint>
+</joint> -->
 <xacro:include filename="$(find drone_frame_description)/urdf/arm.xacro" />
 <xacro:include filename="$(find drone_frame_description)/urdf/coaxial_holder.xacro" />

Commit message: made the ft sensor working

File: drone_frame_description/urdf/drone_frame.xacro (robot description, xacro)
@@ -23,5 +23,5 @@
   </collision>
 </link>
-<!-- <link name="controller">
+<link name="controller">
   <inertial>
     <origin xyz="0.029999999999999964 0.0075 -0.08999999999999991" rpy="0 0 0"/>
@@ -42,6 +42,56 @@
     </geometry>
   </collision>
-</link>
-<joint name="rigid_29" type="fixed">
+  <gazebo>
+    <sensor name="imu_sensor" type="imu"> <!-- IMU Sensor -->
+      <always_on>true</always_on>
+      <update_rate>100</update_rate>
+      <visualize>true</visualize>
+      <topic>imu_data</topic>
+      <imu>
+        <angular_velocity>
+          <x>
+            <noise type="gaussian">
+              <mean>0.0</mean>
+              <stddev>2e-4</stddev>
+            </noise>
+          </x>
+          <y>
+            <noise type="gaussian">
+              <mean>0.0</mean>
+              <stddev>2e-4</stddev>
+            </noise>
+          </y>
+          <z>
+            <noise type="gaussian">
+              <mean>0.0</mean>
+              <stddev>2e-4</stddev>
+            </noise>
+          </z>
+        </angular_velocity>
+        <linear_acceleration>
+          <x>
+            <noise type="gaussian">
+              <mean>0.0</mean>
+              <stddev>1.7e-2</stddev>
+            </noise>
+          </x>
+          <y>
+            <noise type="gaussian">
+              <mean>0.0</mean>
+              <stddev>1.7e-2</stddev>
+            </noise>
+          </y>
+          <z>
+            <noise type="gaussian">
+              <mean>0.0</mean>
+              <stddev>1.7e-2</stddev>
+            </noise>
+          </z>
+        </linear_acceleration>
+      </imu>
+    </sensor>
+  </gazebo>
+</link>
+<joint name="controller_joint" type="fixed">
   <origin xyz="0.0 0.04 0.15" rpy="0 0 0"/>
   <parent link="base_link"/>
@@ -68,5 +118,5 @@
   </collision>
 </link>
-<joint name="rigid_30" type="fixed">
+<joint name="wifi_joint" type="fixed">
   <origin xyz="-0.055 0.04 0.2" rpy="0 0 0"/>
   <parent link="base_link"/>
@@ -92,6 +142,27 @@
     </geometry>
   </collision>
-</link>
-<joint name="rigid_31" type="fixed">
+  <gazebo>
+    <sensor name="camera_front" type="camera"> <!-- Camera Sensor -->
+      <pose>0 0 0.1 0 0 0</pose> <!-- relative to base_link: x, y, z, roll, pitch, yaw -->
+      <always_on>true</always_on>
+      <topic>camera_info</topic>
+      <visualize>true</visualize>
+      <camera>
+        <horizontal_fov>1.047</horizontal_fov> <!-- ~60 degrees -->
+        <image>
+          <width>640</width>
+          <height>480</height>
+          <format>R8G8B8</format>
+        </image>
+        <clip>
+          <near>0.01</near>
+          <far>100</far>
+        </clip>
+      </camera>
+      <update_rate>30</update_rate>
+    </sensor>
+  </gazebo>
+</link>
+<joint name="camera_joint" type="fixed">
   <origin xyz="0.0 0.0 0.15" rpy="0 0 0"/>
   <parent link="base_link"/>
@@ -118,5 +189,5 @@
   </collision>
 </link>
-<joint name="rigid_32" type="fixed">
+<joint name="battery_joint" type="fixed">
   <origin xyz="0.0 0.04 0.0" rpy="0 0 0"/>
   <parent link="base_link"/>
@@ -142,6 +213,16 @@
     </geometry>
   </collision>
-</link>
-<joint name="rigid_33" type="fixed">
+  <gazebo>
+    <sensor name="gps_sensor" type="gps">
+      <pose>0 0 0 0 0 0</pose>
+      <gps>
+        <horizontal_accuracy>0.5</horizontal_accuracy>
+        <vertical_accuracy>1.0</vertical_accuracy>
+        <satellite_count>8</satellite_count>
+      </gps>
+    </sensor>
+  </gazebo>
+</link>
+<joint name="gps_joint" type="fixed">
   <origin xyz="-0.055 0.04 -0.2" rpy="0 0 0"/>
   <parent link="base_link"/>
@@ -168,9 +249,9 @@
   </collision>
 </link>
-<joint name="rigid_34" type="fixed">
+<joint name="testing_probe_joint" type="fixed">
   <origin xyz="0.0 0.02 0.15" rpy="0 0 0"/>
   <parent link="base_link"/>
   <child link="testing_probe"/>
-</joint> -->
+</joint>
 <xacro:include filename="$(find drone_frame_description)/urdf/arm.xacro" />
 <xacro:include filename="$(find drone_frame_description)/urdf/coaxial_holder.xacro" />

File: drone_frame_description/urdf/thruster.xacro (robot description, xacro)
@@ -32,5 +32,4 @@
         <measure_direction>child_to_parent</measure_direction>
       </force_torque>
-      <plugin name="ignition::gazebo::systems::ForceTorque" filename="libignition-gazebo-forcetorque-system.so"/>
     </sensor>
   </gazebo>
